File: mcpcb_11led.kicad_pcb (KiCad board)
At the start: 2 copper layers, 50 x 50 mm, 17 parts

Commit message: fix alignment
Routing:
- net N3: track 14.7 -> 22.2 mm
- net N7: track 12.7 -> 17.2 mm
Changed lines of the file:
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@@
 	(segment
 		(start 35.4 14)
-		(end 39 14)
+		(end 43.5 14)
 		(width 0.4)
 		(layer "F.Cu")
@@
 	)
 	(segment
-		(start 39 14)
+		(start 43.5 14)
+		(end 43.5 25)
+		(width 0.4)
+		(layer "F.Cu")
+		(net "N3")
+	)
+	(segment
+		(start 43.5 25)
 		(end 40.4 25)
 		(width 0.4)
@@
 	)
 	(segment
-		(start 8 25)
+		(start 6.5 36)
 		(end 9.6 36)
 		(width 0.4)
@@
 	)
 	(segment
-		(start 9.6 25)
-		(end 8 25)
+		(start 6.5 25)
+		(end 6.5 36)
 		(width 0.4)
 		(layer "F.Cu")
+		(net "N7")
+	)
+	(segment
+		(start 9.6 25)
+		(end 6.5 25)
+		(width 0.4)
+		(layer "F.Cu")
